Commit message: Fixed up some launch files

File: description/robot_core.xacro (robot description, xacro)
@@ -68,5 +68,5 @@
 			<origin xyz="${chassis_length/2} 0 0" rpy="0 0 0"/>
 		</xacro:inertial_box>
-    	</link>
+    </link>
 	<!-- Left wheel -->
 	<joint name ="left_wheel_joint" type="continuous">

File: description/ros2_control.xacro (robot description, xacro)
@@ -4,9 +4,9 @@
         <ros2_control name="RealRobot" type="system">
             <hardware>
-                <plugin>diffdrive_arduino/DiffDriveArduino</plugin>
+                <plugin>diffdrive_arduino/DiffDriveArduinoHardware</plugin>
                 <param name="left_wheel_name">left_wheel_joint</param>
                 <param name="right_wheel_name">right_wheel_joint</param>
                 <param name="loop_rate">30</param>
-                <param name="device">/usb-1a86_USB_Serial-if00-port0</param>
+                <param name="device">/dev/serial/by-id/usb-1a86_USB_Serial-if00-port0</param>
                 <param name="baud_rate">57600</param>
                 <param name="timeout">1000</param>

Commit message: fuck it we ball

File: description/robot_core.xacro (robot description, xacro)
@@ -3,8 +3,8 @@
     <xacro:include filename="inertial_macros.xacro"/>
 	<!-- Variables -->
-	<xacro:property name="chassis_length" value="-0.365"/>
+	<xacro:property name="chassis_length" value="0.365"/>
     <xacro:property name="chassis_width" value="0.305"/>
 	<xacro:property name="chassis_height" value="0.06"/>
-	<xacro:property name="chassis_base_x_offset" value ="0.081"/>
+	<xacro:property name="chassis_base_x_offset" value ="-0.081"/>
 	<xacro:property name="chassis_base_y_offset" value ="0"/>
 	<xacro:property name="chassis_base_z_offset" value ="0.028"/>
@@ -17,5 +17,5 @@
     <xacro:property name="wheel_offset_z" value="0"/>
     <xacro:property name="caster_wheel_mass" value="0.5"/>
-	<xacro:property name="caster_wheel_offset_x" value="-0.33175"/>
+	<xacro:property name="caster_wheel_offset_x" value="0.33175"/>
 	<xacro:property name="caster_wheel_offset_y" value="0.11925"/>
     <xacro:property name="caster_wheel_offset_z" value="-${chassis_base_z_offset}"/>

Commit message: No more Bryant haha

File: description/robot_core.xacro (robot description, xacro)
@@ -6,5 +6,5 @@
     <xacro:property name="chassis_width" value="0.305"/>
 	<xacro:property name="chassis_height" value="0.06"/>
-	<xacro:property name="chassis_base_x_offset" value ="-0.089"/>
+	<xacro:property name="chassis_base_x_offset" value ="-0.081"/>
 	<xacro:property name="chassis_base_y_offset" value ="0"/>
 	<xacro:property name="chassis_base_z_offset" value ="0.028"/>
