Commit message: added sensors into the nav stack

File: description/depth_camera.xacro (robot description, xacro)
@@ -2,7 +2,7 @@
 <robot xmlns:xacro="http://www.ros.org/wiki/xacro">
 	<joint name="camera_joint" type="fixed">
-		<parent link="chassis"/>
+		<parent link="r2d2_chassis"/>
 		<child link="camera_link"/>
-		<origin xyz="${0.365 +0.01} 0 0.03" rpy="0 0 0"/>
+		<origin xyz="${(0.2315 +0.01)} 0 ${0.47527/2}" rpy="0 0 0"/>
 	</joint>
 	<link name="camera_link">

File: description/imu.xacro (robot description, xacro)
@@ -2,7 +2,7 @@
 <robot xmlns:xacro="http://www.ros.org/wiki/xacro">
 	<joint name="imu_joint" type="fixed">
-		<parent link="chassis"/>
+		<parent link="camera_link"/>
 		<child link="imu_link"/>
-		<origin xyz="${0.365 +0.01} 0 0.03" rpy="0 0 0"/>
+		<origin xyz="0 0 0" rpy="0 0 0"/>
 	</joint>
 	<link name="imu_link">
@@ -19,10 +19,4 @@
 		</collision>
 	</link>
-	<joint name="imu_sensor_joint" type="fixed">
-		<parent link="imu_link"/>
-		<child link="imu_pos_link"/>
-		<origin xyz="0 0 0" rpy="${-pi/2} 0 ${-pi/2}"/>
-	</joint>
-	<link name="imu_pos_link"></link>
 <gazebo reference ="imu_link">
 	<sensor name="imu_sensor" type="imu">

File: description/robot_core.xacro (robot description, xacro)
@@ -20,4 +20,7 @@
 	<xacro:property name="caster_wheel_offset_y" value="0.11925"/>
     <xacro:property name="caster_wheel_offset_z" value="-${chassis_base_z_offset}"/>
+	<xacro:property name="r2d2_height" value="0.47527"/>
+	<xacro:property name="r2d2_radius" value="0.2315"/>
+	<xacro:property name="r2d2_base_z_offset" value ="0.125038"/>
     <material name="white">
         <color rgba="1 1 1 1" />
@@ -68,4 +71,49 @@
 			<origin xyz="${chassis_length/2} 0 0" rpy="0 0 0"/>
 		</xacro:inertial_box>
+    </link>
+	<!-- R2D2 body -->
+	<joint name="r2d2_body" type="fixed">
+        <parent link="chassis"/>
+        <child link="r2d2_chassis"/>
+		<origin xyz="${chassis_length/2} 0 ${r2d2_base_z_offset + r2d2_height/2}" rpy="0 0 0"/>
+    </joint>
+	<link name="r2d2_chassis">
+		<visual>
+			<origin xyz="0 0 0"/>
+			<geometry>
+				<cylinder radius="${r2d2_radius}" length="${r2d2_height}"/>
+			</geometry>
+			<material name="white"/>
+		</visual>
+		<collision>
+			<geometry>
+				<cylinder radius="${r2d2_radius}" length="${r2d2_height}"/>
+			</geometry>
+		</collision>
+		<xacro:inertial_cylinder mass="0.0001" radius="${r2d2_radius}" length="${r2d2_height}">
+			<origin xyz="0 0 0" rpy="0 0 0"/>
+		</xacro:inertial_cylinder>
+    </link>
+	<joint name="r2d2_head" type="fixed">
+        <parent link="r2d2_chassis"/>
+        <child link="head"/>
+		<origin xyz="0 0 ${r2d2_height/2}" rpy="0 0 0"/>
+    </joint>
+	<link name="head">
+		<visual>
+			<origin xyz="0 0 0"/>
+			<geometry>
+				<sphere radius="${r2d2_radius}"/>
+			</geometry>
+			<material name="white"/>
+		</visual>
+		<collision>
+			<geometry>
+				<sphere radius="${r2d2_radius}"/>
+			</geometry>
+		</collision>
+		<xacro:inertial_sphere mass="0.0001" radius="${r2d2_radius}">
+			<origin xyz="0 0 0" rpy="0 0 0"/>
+		</xacro:inertial_sphere>
     </link>
 	<!-- Left wheel -->

File: description/us_sensor.xacro (robot description, xacro)
@@ -2,30 +2,206 @@
 <robot xmlns:xacro="http://www.ros.org/wiki/xacro">
 	<joint name="us1_joint" type="fixed">
-		<parent link="chassis"/>
+		<parent link="r2d2_chassis"/>
 		<child link="us1_link"/>
-		<origin xyz="0 0 0" rpy="0 0 0"/>
+		<origin xyz="${(0.2315 +0.01)} 0 0" rpy="0 0 0"/>
 	</joint>
 	<link name="us1_link">
-	</link>
+		<origin xyz="0 0 0" rpy="0 0 0"/>
+	</link>
+	<gazebo reference="us1_link">
+		<sensor name="us_ultrasound_1" type="ray">
+			<always_on>true</always_on>
+			<visualize>true</visualize>
+			<pose>0.0 0 0.0 0 0 0</pose>
+			<update_rate>50</update_rate>
+			<ray>
+				<scan>
+					<horizontal>
+						<samples>5</samples>
+						<resolution>1.0</resolution>
+						<min_angle>-0.18</min_angle>
+						<max_angle>0.18</max_angle>
+					</horizontal>
+					<vertical>
+						<samples>5</samples>
+						<resolution>1.0</resolution>
+						<min_angle>-0.01</min_angle>
+						<max_angle>0.01</max_angle>
+					</vertical>
+				</scan>
+				<range>
+					<min>0.02</min>
+					<max>4</max>
+					<resolution>0.01</resolution>
+				</range>
+				<noise>
+					<type>gaussian</type>
+					<mean>0.0</mean>
+					<stddev>0.01</stddev>
+				</noise>
+			</ray>
+			 <plugin name="bytes_ultrasound1" filename="libgazebo_ros_ray_sensor.so">
+				<ros>
+					<remapping>~/out:=Us1/Range</remapping>
+				</ros>
+				<output_type>sensor_msgs/Range</output_type>
+				<radiation_type>ultrasound</radiation_type>
+				<frame_name>us1_link</frame_name>
+			</plugin>
+		</sensor>
+		<material>Gazebo/Blue</material>
+	</gazebo>
 	<joint name="us2_joint" type="fixed">
-		<parent link="chasis"/>
+		<parent link="r2d2_chassis"/>
 		<child link="us2_link"/>
-		<origin xyz="0 0 0" rpy="0 0 0"/>
+		<origin xyz="0 ${-(0.2315 +0.01)} 0" rpy="0 0 ${-pi/2}"/>
 	</joint>
 	<link name="us2_link">
-	</link>
+		<origin xyz="0 0 0" rpy="0 0 0"/>
+	</link>
+	<gazebo reference="us2_link">
+		<sensor name="us_ultrasound_2" type="ray">
+			<always_on>true</always_on>
+			<visualize>true</visualize>
+			<pose>0.0 0 0.0 0 0 0</pose>
+			<update_rate>50</update_rate>
+			<ray>
+				<scan>
+					<horizontal>
+						<samples>5</samples>
+						<resolution>1.0</resolution>
+						<min_angle>-0.18</min_angle>
+						<max_angle>0.18</max_angle>
+					</horizontal>
+					<vertical>
+						<samples>5</samples>
+						<resolution>1.0</resolution>
+						<min_angle>-0.01</min_angle>
+						<max_angle>0.01</max_angle>
+					</vertical>
+				</scan>
+				<range>
+					<min>0.02</min>
+					<max>4</max>
+					<resolution>0.01</resolution>
+				</range>
+				<noise>
+					<type>gaussian</type>
+					<mean>0.0</mean>
+					<stddev>0.01</stddev>
+				</noise>
+			</ray>
+			 <plugin name="bytes_ultrasound2" filename="libgazebo_ros_ray_sensor.so">
+				<ros>
+					<remapping>~/out:=Us2/Range</remapping>
+				</ros>
+				<output_type>sensor_msgs/Range</output_type>
+				<radiation_type>ultrasound</radiation_type>
+				<frame_name>us2_link</frame_name>
+			</plugin>
+		</sensor>
+		<material>Gazebo/Blue</material>
+	</gazebo>
 	<joint name="us3_joint" type="fixed">
-		<parent link="chassis"/>
+		<parent link="r2d2_chassis"/>
 		<child link="us3_link"/>
-		<origin xyz="0 0 0" rpy="0 0 0"/>
+		<origin xyz="${-(0.2315 +0.01)} 0 0" rpy="0 0 ${-pi}"/>
 	</joint>
 	<link name="us3_link">
-	</link>
+		<origin xyz="0 0 0" rpy="0 0 0"/>
+	</link>
+	<gazebo reference="us3_link">
+		<sensor name="us_ultrasound_3" type="ray">
+			<always_on>true</always_on>
+			<visualize>true</visualize>
+			<pose>0.0 0 0.0 0 0 0</pose>
+			<update_rate>50</update_rate>
+			<ray>
+				<scan>
+					<horizontal>
+						<samples>5</samples>
+						<resolution>1.0</resolution>
+						<min_angle>-0.18</min_angle>
+						<max_angle>0.18</max_angle>
+					</horizontal>
+					<vertical>
+						<samples>5</samples>
+						<resolution>1.0</resolution>
+						<min_angle>-0.01</min_angle>
+						<max_angle>0.01</max_angle>
+					</vertical>
+				</scan>
+				<range>
+					<min>0.02</min>
+					<max>4</max>
+					<resolution>0.01</resolution>
+				</range>
+				<noise>
+					<type>gaussian</type>
+					<mean>0.0</mean>
+					<stddev>0.01</stddev>
+				</noise>
+			</ray>
+			 <plugin name="bytes_ultrasound3" filename="libgazebo_ros_ray_sensor.so">
+				<ros>
+					<remapping>~/out:=Us3/Range</remapping>
+				</ros>
+				<output_type>sensor_msgs/Range</output_type>
+				<radiation_type>ultrasound</radiation_type>
+				<frame_name>us3_link</frame_name>
+			</plugin>
+		</sensor>
+		<material>Gazebo/Blue</material>
+	</gazebo>
 	<joint name="us4_joint" type="fixed">
-		<parent link="chasis"/>
+		<parent link="r2d2_chassis"/>
 		<child link="us4_link"/>
-		<origin xyz="0 0 0" rpy="0 0 0"/>
+		<origin xyz="0 ${(0.2315 +0.01)} 0" rpy="0 0 ${pi/2}"/>
 	</joint>
 	<link name="us4_link">
-	</link>
+		<origin xyz="0 0 0" rpy="0 0 0"/>
+	</link>
+	<gazebo reference="us4_link">
+		<sensor name="us_ultrasound_4" type="ray">
+			<always_on>true</always_on>
+			<visualize>true</visualize>
+			<pose>0.0 0 0.0 0 0 0</pose>
+			<update_rate>50</update_rate>
+			<ray>
+				<scan>
+					<horizontal>
+						<samples>5</samples>
+						<resolution>1.0</resolution>
+						<min_angle>-0.18</min_angle>
+						<max_angle>0.18</max_angle>
+					</horizontal>
+					<vertical>
+						<samples>5</samples>
+						<resolution>1.0</resolution>
+						<min_angle>-0.01</min_angle>
+						<max_angle>0.01</max_angle>
+					</vertical>
+				</scan>
+				<range>
+					<min>0.02</min>
+					<max>4</max>
+					<resolution>0.01</resolution>
+				</range>
+				<noise>
+					<type>gaussian</type>
+					<mean>0.0</mean>
+					<stddev>0.01</stddev>
+				</noise>
+			</ray>
+			 <plugin name="bytes_ultrasound4" filename="libgazebo_ros_ray_sensor.so">
+				<ros>
+					<remapping>~/out:=Us4/Range</remapping>
+				</ros>
+				<output_type>sensor_msgs/Range</output_type>
+				<radiation_type>ultrasound</radiation_type>
+				<frame_name>us4_link</frame_name>
+			</plugin>
+		</sensor>
+		<material>Gazebo/Blue</material>
+	</gazebo>
 </robot>

Commit message: fixed urdf

File: description/depth_camera.xacro (robot description, xacro)
@@ -4,5 +4,5 @@
 		<parent link="r2d2_chassis"/>
 		<child link="camera_link"/>
-		<origin xyz="${(0.2315 +0.01)} 0 ${0.47527/2}" rpy="0 0 0"/>
+		<origin xyz="${(0.2315)} 0 ${0.47527/2}" rpy="0 0 0"/>
 	</joint>
 	<link name="camera_link">

File: description/robot_core.xacro (robot description, xacro)
@@ -6,5 +6,5 @@
     <xacro:property name="chassis_width" value="0.305"/>
 	<xacro:property name="chassis_height" value="0.06"/>
-	<xacro:property name="chassis_base_x_offset" value ="-0.081"/>
+	<xacro:property name="chassis_base_x_offset" value ="-0.089"/>
 	<xacro:property name="chassis_base_y_offset" value ="0"/>
 	<xacro:property name="chassis_base_z_offset" value ="0.028"/>

File: description/us_sensor.xacro (robot description, xacro)
@@ -2,7 +2,7 @@
 <robot xmlns:xacro="http://www.ros.org/wiki/xacro">
 	<joint name="us1_joint" type="fixed">
-		<parent link="r2d2_chassis"/>
+		<parent link="camera_link"/>
 		<child link="us1_link"/>
-		<origin xyz="${(0.2315 +0.01)} 0 0" rpy="0 0 0"/>
+		<origin xyz="0 0 -0.038" rpy="0 0 0"/>
 	</joint>
 	<link name="us1_link">
@@ -55,5 +55,5 @@
 		<parent link="r2d2_chassis"/>
 		<child link="us2_link"/>
-		<origin xyz="0 ${-(0.2315 +0.01)} 0" rpy="0 0 ${-pi/2}"/>
+		<origin xyz="0 ${-(0.2315 +0.01)} -0.15" rpy="0 0 ${-pi/2}"/>
 	</joint>
 	<link name="us2_link">
@@ -106,5 +106,5 @@
 		<parent link="r2d2_chassis"/>
 		<child link="us3_link"/>
-		<origin xyz="${-(0.2315 +0.01)} 0 0" rpy="0 0 ${-pi}"/>
+		<origin xyz="${(0.2315)} 0 ${-0.47527/2+0.15}" rpy="0 0 0"/>
 	</joint>
 	<link name="us3_link">
@@ -157,5 +157,5 @@
 		<parent link="r2d2_chassis"/>
 		<child link="us4_link"/>
-		<origin xyz="0 ${(0.2315 +0.01)} 0" rpy="0 0 ${pi/2}"/>
+		<origin xyz="0 ${(0.2315 +0.01)} -0.15" rpy="0 0 ${pi/2}"/>
 	</joint>
 	<link name="us4_link">

Commit message: pain

File: description/depth_camera.xacro (robot description, xacro)
@@ -4,5 +4,5 @@
 		<parent link="r2d2_chassis"/>
 		<child link="camera_link"/>
-		<origin xyz="${(0.2315)} 0 ${0.47527/2}" rpy="0 0 0"/>
+		<origin xyz="${(0.2315)} 0 ${0.47527/2+0.038}" rpy="0 0 0"/>
 	</joint>
 	<link name="camera_link">
@@ -39,9 +39,12 @@
                 </image>
                 <clip>
-                    <near>0.05</near>
+                    <near>0.005</near>
                     <far>8.0</far>
                 </clip>
             </camera>
             <plugin name="camera_controller" filename="libgazebo_ros_camera.so">
+				<ros>
+					<remapping>/camera/points:=/camera/depth/color/points</remapping>
+				</ros>
 				<frame_name>camera_link_optical</frame_name>
 				<min_depth>0.1</min_depth>

File: description/imu.xacro (robot description, xacro)
@@ -23,5 +23,5 @@
 		<plugin filename="libgazebo_ros_imu_sensor.so" name="imu_plugin">
 		<ros>
-			<remapping>~/out:=imu</remapping>
+			<remapping>~/out:=camera/imu</remapping>
 		</ros>
 		<initial_orientation_as_reference>false</initial_orientation_as_reference>

File: description/robot_core.xacro (robot description, xacro)
@@ -86,9 +86,9 @@
 			<material name="white"/>
 		</visual>
-		<collision>
+		<!--collision>
 			<geometry>
 				<cylinder radius="${r2d2_radius}" length="${r2d2_height}"/>
 			</geometry>
-		</collision>
+		</collision-->
 		<xacro:inertial_cylinder mass="0.0001" radius="${r2d2_radius}" length="${r2d2_height}">
 			<origin xyz="0 0 0" rpy="0 0 0"/>
@@ -108,9 +108,9 @@
 			<material name="white"/>
 		</visual>
-		<collision>
+		<!--collision>
 			<geometry>
 				<sphere radius="${r2d2_radius}"/>
 			</geometry>
-		</collision>
+		</collision-->
 		<xacro:inertial_sphere mass="0.0001" radius="${r2d2_radius}">
 			<origin xyz="0 0 0" rpy="0 0 0"/>

Commit message: imu fixes

File: description/depth_camera.xacro (robot description, xacro)
@@ -46,4 +46,7 @@
 				<ros>
 					<remapping>/camera/points:=/camera/depth/color/points</remapping>
+					<remapping>/camera/depth/image_raw:=/camera/color/image_raw</remapping>
+					<remapping>/camera/camera_info:=/camera/color/camera_info</remapping>
+					<remapping>/camera/image_raw:=/camera/realigned_depth_to_color/image_raw</remapping>
 				</ros>
 				<frame_name>camera_link_optical</frame_name>

File: description/imu.xacro (robot description, xacro)
@@ -2,5 +2,5 @@
 <robot xmlns:xacro="http://www.ros.org/wiki/xacro">
 	<joint name="imu_joint" type="fixed">
-		<parent link="camera_link_optical"/>
+		<parent link="camera_link"/>
 		<child link="camera_imu_optical_frame"/>
 		<origin xyz="0 0 0" rpy="0 0 0"/>
