Commit message: fixed up lidar urdf

File: description/lidar.xacro (robot description, xacro)
@@ -4,10 +4,10 @@
 		<parent link="chassis"/>
 		<child link="laser_frame"/>
-		<origin xyz="0 0 0.07" rpy="0 0 0"/>
+		<origin xyz="0 0 0.115288" rpy="0 ${pi} 0"/>
 	</joint>
 		<link name="laser_frame">
 			<visual>
 				<geometry>
-					<cylinder radius="0.05" length="0.04"/>
+					<cylinder radius="0.07" length="0.0195"/>
 				</geometry>
 				<material name ="blue"/>
@@ -15,9 +15,9 @@
 			<collision>
 				<geometry>
-					<cylinder radius="0.05" length="0.04"/>
+					<cylinder radius="0.07" length="0.0195"/>
 				</geometry>
 			</collision>
 			<xacro:inertial_cylinder mass="0.1" radius="0.05" length="0.04">
-				<origin xyz="0 0 0.07" rpy="0 0 0"/>
+				<origin xyz="0 0 0.07" rpy="0 ${pi} 0"/>
 			</xacro:inertial_cylinder>
 		</link>

Commit message: lidar

File: description/lidar.xacro (robot description, xacro)
@@ -4,5 +4,5 @@
 		<parent link="chassis"/>
 		<child link="laser_frame"/>
-		<origin xyz="0 0 0.115288" rpy="0 ${pi} 0"/>
+		<origin xyz="0.365 0 0.115288" rpy="0 ${pi} 0"/>
 	</joint>
 		<link name="laser_frame">
@@ -19,5 +19,5 @@
 			</collision>
 			<xacro:inertial_cylinder mass="0.1" radius="0.05" length="0.04">
-				<origin xyz="0 0 0.07" rpy="0 ${pi} 0"/>
+				<origin xyz="0.365 0 0.115288" rpy="0 ${pi} 0"/>
 			</xacro:inertial_cylinder>
 		</link>

Commit message: changed urdf

File: description/lidar.xacro (robot description, xacro)
@@ -4,5 +4,5 @@
 		<parent link="chassis"/>
 		<child link="laser_frame"/>
-		<origin xyz="0.365 0 0.115288" rpy="0 ${pi} 0"/>
+		<origin xyz="0 0 0.115288" rpy="0 ${pi} 0"/>
 	</joint>
 		<link name="laser_frame">
@@ -19,5 +19,5 @@
 			</collision>
 			<xacro:inertial_cylinder mass="0.1" radius="0.05" length="0.04">
-				<origin xyz="0.365 0 0.115288" rpy="0 ${pi} 0"/>
+				<origin xyz="0 0 0.115288" rpy="0 ${pi} 0"/>
 			</xacro:inertial_cylinder>
 		</link>

File: description/robot_core.xacro (robot description, xacro)
@@ -3,8 +3,8 @@
     <xacro:include filename="inertial_macros.xacro"/>
 	<!-- Variables -->
-	<xacro:property name="chassis_length" value="0.365"/>
+	<xacro:property name="chassis_length" value="-0.365"/>
     <xacro:property name="chassis_width" value="0.305"/>
 	<xacro:property name="chassis_height" value="0.06"/>
-	<xacro:property name="chassis_base_x_offset" value ="-0.081"/>
+	<xacro:property name="chassis_base_x_offset" value ="0.081"/>
 	<xacro:property name="chassis_base_y_offset" value ="0"/>
 	<xacro:property name="chassis_base_z_offset" value ="0.028"/>
@@ -17,5 +17,5 @@
     <xacro:property name="wheel_offset_z" value="0"/>
     <xacro:property name="caster_wheel_mass" value="0.5"/>
-	<xacro:property name="caster_wheel_offset_x" value="0.33175"/>
+	<xacro:property name="caster_wheel_offset_x" value="-0.33175"/>
 	<xacro:property name="caster_wheel_offset_y" value="0.11925"/>
     <xacro:property name="caster_wheel_offset_z" value="-${chassis_base_z_offset}"/>

Commit message: fuck balling

File: description/lidar.xacro (robot description, xacro)
@@ -4,5 +4,5 @@
 		<parent link="chassis"/>
 		<child link="laser_frame"/>
-		<origin xyz="0 0 0.115288" rpy="0 ${pi} 0"/>
+		<origin xyz="0 0 0.115288" rpy="0 ${pi} ${pi}"/>
 	</joint>
 		<link name="laser_frame">
@@ -19,5 +19,5 @@
 			</collision>
 			<xacro:inertial_cylinder mass="0.1" radius="0.05" length="0.04">
-				<origin xyz="0 0 0.115288" rpy="0 ${pi} 0"/>
+				<origin xyz="0 0 0.115288" rpy="0 ${pi} ${pi}"/>
 			</xacro:inertial_cylinder>
 		</link>

Commit message: fuck balling

File: description/lidar.xacro (robot description, xacro)
@@ -4,5 +4,5 @@
 		<parent link="chassis"/>
 		<child link="laser_frame"/>
-		<origin xyz="0 0 0.115288" rpy="0 ${pi} ${pi}"/>
+		<origin xyz="0.365 0 0.115288" rpy="0 ${pi} 0"/>
 	</joint>
 		<link name="laser_frame">
@@ -19,5 +19,5 @@
 			</collision>
 			<xacro:inertial_cylinder mass="0.1" radius="0.05" length="0.04">
-				<origin xyz="0 0 0.115288" rpy="0 ${pi} ${pi}"/>
+				<origin xyz="0.365 0 0.115288" rpy="0 ${pi} 0"/>
 			</xacro:inertial_cylinder>
 		</link>

Commit message: ligma balls

File: description/lidar.xacro (robot description, xacro)
@@ -4,5 +4,5 @@
 		<parent link="chassis"/>
 		<child link="laser_frame"/>
-		<origin xyz="0.365 0 0.115288" rpy="0 ${pi} 0"/>
+		<origin xyz="-0.060 0 0.115288" rpy="0 ${pi} 0"/>
 	</joint>
 		<link name="laser_frame">

File: description/robot_core.xacro (robot description, xacro)
@@ -3,19 +3,19 @@
     <xacro:include filename="inertial_macros.xacro"/>
 	<!-- Variables -->
-	<xacro:property name="chassis_length" value="0.365"/>
+	<xacro:property name="chassis_length" value="-0.365"/>
     <xacro:property name="chassis_width" value="0.305"/>
 	<xacro:property name="chassis_height" value="0.06"/>
-	<xacro:property name="chassis_base_x_offset" value ="-0.081"/>
+	<xacro:property name="chassis_base_x_offset" value ="0.060"/>
 	<xacro:property name="chassis_base_y_offset" value ="0"/>
 	<xacro:property name="chassis_base_z_offset" value ="0.028"/>
     <xacro:property name="chassis_mass" value="1.0"/>
-    <xacro:property name="wheel_radius" value="0.04175"/>
-    <xacro:property name="wheel_thickness" value="0.04977"/>
+    <xacro:property name="wheel_radius" value="0.08255"/>
+    <xacro:property name="wheel_thickness" value="0.04635"/>
     <xacro:property name="wheel_mass" value="0.5"/>
     <xacro:property name="wheel_offset_x" value="0"/>
-    <xacro:property name="wheel_offset_y" value="0.01578"/>
+    <xacro:property name="wheel_offset_y" value="0.023"/>
     <xacro:property name="wheel_offset_z" value="0"/>
     <xacro:property name="caster_wheel_mass" value="0.5"/>
-	<xacro:property name="caster_wheel_offset_x" value="0.33175"/>
+	<xacro:property name="caster_wheel_offset_x" value="-0.33175"/>
 	<xacro:property name="caster_wheel_offset_y" value="0.11925"/>
     <xacro:property name="caster_wheel_offset_z" value="-${chassis_base_z_offset}"/>
