Commit message: FIXED RANGE SENSORS ETC

File: description/imu.xacro (robot description, xacro)
@@ -20,4 +20,5 @@
 	</link>
 <gazebo reference ="imu_link">
+	<gravity>true</gravity>
 	<sensor name="imu_sensor" type="imu">
 		<plugin filename="libgazebo_ros_imu_sensor.so" name="imu_plugin">
@@ -25,5 +26,10 @@
 			<remapping>~/out:=camera/imu</remapping>
 		</ros>
-		<initial_orientation_as_reference>false</initial_orientation_as_reference>
+		<always_on>true</always_on>
+      	<update_rate>100</update_rate>
+      	<visualize>true</visualize>
+		<bodyName>imu_link</bodyName>
+        <updateRateHZ>10.0</updateRateHZ>
+        <gaussianNoise>0.0</gaussianNoise>
 		<frame_name>imu_link</frame_name>
 		</plugin>
@@ -31,58 +37,5 @@
 		<update_rate>100</update_rate>
 		<visualize>true</visualize>
-		<imu>
-		<angular_velocity>
-			<x>
-			<noise type="gaussian">
-				<mean>0.0</mean>
-				<stddev>2e-4</stddev>
-				<bias_mean>0.0000075</bias_mean>
-				<bias_stddev>0.0000008</bias_stddev>
-			</noise>
-			</x>
-			<y>
-			<noise type="gaussian">
-				<mean>0.0</mean>
-				<stddev>2e-4</stddev>
-				<bias_mean>0.0000075</bias_mean>
-				<bias_stddev>0.0000008</bias_stddev>
-			</noise>
-			</y>
-			<z>
-			<noise type="gaussian">
-				<mean>0.0</mean>
-				<stddev>2e-4</stddev>
-				<bias_mean>0.0000075</bias_mean>
-				<bias_stddev>0.0000008</bias_stddev>
-			</noise>
-			</z>
-		</angular_velocity>
-		<linear_acceleration>
-			<x>
-			<noise type="gaussian">
-				<mean>0.0</mean>
-				<stddev>1.7e-2</stddev>
-				<bias_mean>0.1</bias_mean>
-				<bias_stddev>0.001</bias_stddev>
-			</noise>
-			</x>
-			<y>
-			<noise type="gaussian">
-				<mean>0.0</mean>
-				<stddev>1.7e-2</stddev>
-				<bias_mean>0.1</bias_mean>
-				<bias_stddev>0.001</bias_stddev>
-			</noise>
-			</y>
-			<z>
-			<noise type="gaussian">
-				<mean>0.0</mean>
-				<stddev>1.7e-2</stddev>
-				<bias_mean>0.1</bias_mean>
-				<bias_stddev>0.001</bias_stddev>
-			</noise>
-			</z>
-		</linear_acceleration>
-		</imu>
+		<initialOrientationAsReference>false</initialOrientationAsReference>
 	</sensor>
 </gazebo>

File: description/lidar.xacro (robot description, xacro)
@@ -26,5 +26,5 @@
         <sensor name="laser" type="ray">
             <pose> 0 0 0 0 0 0 </pose>
-            <visualize>true</visualize>
+            <visualize>false</visualize>
             <update_rate>10</update_rate>
             <ray>

File: description/robot_core.xacro (robot description, xacro)
@@ -86,9 +86,9 @@
 			<material name="white"/>
 		</visual>
-		<!--collision>
+		<collision>
 			<geometry>
 				<cylinder radius="${r2d2_radius}" length="${r2d2_height}"/>
 			</geometry>
-		</collision-->
+		</collision>
 		<xacro:inertial_cylinder mass="0.0001" radius="${r2d2_radius}" length="${r2d2_height}">
 			<origin xyz="0 0 0" rpy="0 0 0"/>
@@ -108,9 +108,9 @@
 			<material name="white"/>
 		</visual>
-		<!--collision>
+		<collision>
 			<geometry>
 				<sphere radius="${r2d2_radius}"/>
 			</geometry>
-		</collision-->
+		</collision>
 		<xacro:inertial_sphere mass="0.0001" radius="${r2d2_radius}">
 			<origin xyz="0 0 0" rpy="0 0 0"/>

File: description/us_sensor.xacro (robot description, xacro)
@@ -12,5 +12,5 @@
 		<sensor name="us_ultrasound_1" type="ray">
 			<always_on>true</always_on>
-			<visualize>true</visualize>
+			<visualize>false</visualize>
 			<pose>0.0 0 0.0 0 0 0</pose>
 			<update_rate>50</update_rate>
@@ -63,5 +63,5 @@
 		<sensor name="us_ultrasound_2" type="ray">
 			<always_on>true</always_on>
-			<visualize>true</visualize>
+			<visualize>false</visualize>
 			<pose>0.0 0 0.0 0 0 0</pose>
 			<update_rate>50</update_rate>
@@ -114,5 +114,5 @@
 		<sensor name="us_ultrasound_3" type="ray">
 			<always_on>true</always_on>
-			<visualize>true</visualize>
+			<visualize>false</visualize>
 			<pose>0.0 0 0.0 0 0 0</pose>
 			<update_rate>50</update_rate>
@@ -165,5 +165,5 @@
 		<sensor name="us_ultrasound_4" type="ray">
 			<always_on>true</always_on>
-			<visualize>true</visualize>
+			<visualize>false</visualize>
 			<pose>0.0 0 0.0 0 0 0</pose>
 			<update_rate>50</update_rate>

Commit message: imu?

File: description/imu.xacro (robot description, xacro)
@@ -2,9 +2,9 @@
 <robot xmlns:xacro="http://www.ros.org/wiki/xacro">
 	<joint name="imu_joint" type="fixed">
-		<parent link="camera_link"/>
-		<child link="imu_link"/>
+		<parent link="camera_link_optical"/>
+		<child link="camera_imu_optical_frame"/>
 		<origin xyz="0 0 0" rpy="0 0 0"/>
 	</joint>
-	<link name="imu_link">
+	<link name="camera_imu_optical_frame">
 		<visual>
 			<geometry>
@@ -19,5 +19,5 @@
 		</collision>
 	</link>
-<gazebo reference ="imu_link">
+<gazebo reference ="camera_imu_optical_frame">
 	<gravity>true</gravity>
 	<sensor name="imu_sensor" type="imu">
@@ -29,8 +29,8 @@
       	<update_rate>100</update_rate>
       	<visualize>true</visualize>
-		<bodyName>imu_link</bodyName>
+		<bodyName>camera_imu_optical_frame</bodyName>
         <updateRateHZ>10.0</updateRateHZ>
         <gaussianNoise>0.0</gaussianNoise>
-		<frame_name>imu_link</frame_name>
+		<frame_name>camera_imu_optical_frame</frame_name>
 		</plugin>
 		<always_on>true</always_on>

File: description/ros2_control.xacro (robot description, xacro)
@@ -9,4 +9,5 @@
                 <param name="loop_rate">30</param>
                 <!--param name="device">/dev/serial/by-id/usb-Arduino__www.arduino.cc__0043_9593132313235151F031-if00</param-->
+                <!--param name="device">/dev/ttyUSB0</param-->
                 <param name="device">/dev/serial/by-id/usb-1a86_USB_Serial-if00-port0</param>
                 <param name="baud_rate">57600</param>

Commit message: imu

File: description/imu.xacro (robot description, xacro)
@@ -2,5 +2,5 @@
 <robot xmlns:xacro="http://www.ros.org/wiki/xacro">
 	<joint name="imu_joint" type="fixed">
-		<parent link="camera_link"/>
+		<parent link="camera_link_optical"/>
 		<child link="camera_imu_optical_frame"/>
 		<origin xyz="0 0 0" rpy="0 0 0"/>
